File: Orb_hw/Orb.kicad_sch (KiCad schematic)
At the start: 73 parts, among them Q1 IRLML6401, Q2 2N7002, Q3 IRF9317, Q4 2N7002, SW1 BUTTON, SW2 BUTTON, SW3 BUTTON

Commit message: + Sent to factory
Parts:
- removed TP1: TESTPOINT, PCB:TESTPOINT_1MM, symbol pcb_details:TESTPOINT
- added HOLE6: HOLE_METALLED, PCB:Hole2d4_out4d4mm, symbol pcb_details:HOLE_METALLED
- added Q5: IRLML6401, SOT:SOT23-3, symbol Transistors_kl:P_3PIN
- added XL5: CONN_1, Connectors:PLS-1Square, symbol Connectors_kl:CONN_1
- ANT1: footprint Antennas:MagicStick -> Antennas:Firefly_868
- HOLE1, HOLE2, HOLE3, HOLE4, HOLE5: footprint PCB:Hole2d4_out4d5mm -> PCB:Hole2d4_out4d4mm
- Logo1: footprint Pictures:Ostranna_8x8 -> Pictures:Ostranna_16d9_13d5
Connections:
- net +BATT: now also Q5.2 (S)
- net GND: now also HOLE6.H, XL5.1 (P1)
- net NPX_PWR: now also Q5.3 (D)
- net at Q2.3 (D), Q3.4 (G), R8.2: now also Q5.1 (G)
- no-connect marks 18 -> 19
Other:
- note added: "Maybe this one is acceptable: 50 mOhm"
